File: CuttingMachine_PCB/Buttons/CutMachine_PCB.kicad_pcb (KiCad board)
At the start: 2 copper layers, 54.9 x 34.3 mm, 10 parts, among them J2 Conn_01x07_Pin, SW3 DOWN

Commit message: Add files via upload
Other:
- outline, holes or cut-outs redrawn
- board text added: "Pips was here"
- board text added: "UtahSaint CutMachineSMD Button PCB"
- board text added: "github.com/utahsaint-org/CutMachineSMD"
