File: CuttingMachine_PCB/Sensor/Sensor.kicad_pcb (KiCad board)
At the start: 2 copper layers, 20 x 25 mm, 4 parts, among them J1 Conn_01x03_Pin

Commit message: Add files via upload
Parts:
- added JP1: SolderJumper_3_Open, Jumper:SolderJumper-3_P2.0mm_Open_TrianglePad1.0x1.5mm_NumberLabels, F.Cu at (141.5, 99.8)
- added R3: 470, Resistor_SMD:R_1206_3216Metric_Pad1.30x1.75mm_HandSolder, F.Cu at (138.2, 95.2)
- R2: renamed from 10KΩ; value 220 -> 2.2k
- renumbered OPT1 to O1, 470Ω to R1
Connections:
- R2 pad 2: Net-(J1-Pin_3) -> Net-(JP1-B)
Routing:
- net Net-(J1-Pin_3): track 17.5 -> 23.9 mm
- net Net-(J1-Pin_2): track 6.55 -> 12.4 mm, vias 0 -> 2
- net Net-(JP1-B): track 0.00 -> 3.59 mm
- net Net-(JP1-A): track 0.00 -> 3.56 mm
- net Net-(O1-E+): track 13.8 -> 14.8 mm
- removed copper zone on B.Cu, net (none)
- removed copper zone on F.Cu, net (none)
Other:
- outline, holes or cut-outs redrawn
- board text added: "POS"
- board text added: "PRS"
- board text added: "UtahSaint CutMachineSMD Sensor PCB"
- board text added: "pips was here"
