File: CuttingMachine_PCB/Sensor/Sensor.kicad_sch (KiCad schematic)
At the start: 4 parts, among them J1 Conn_01x03_Pin

Commit message: Add files via upload
Parts:
- added JP1: SolderJumper_3_Open, Jumper:SolderJumper-3_P2.0mm_Open_TrianglePad1.0x1.5mm_NumberLabels, symbol Jumper:SolderJumper_3_Open
- added R3: 470, Resistor_SMD:R_1206_3216Metric_Pad1.30x1.75mm_HandSolder, symbol Device:R_US
- R2: value 220 -> 2.2k
Connections:
- net at J1.2 (Pin_2), R1.1, R2.1: now also R3.1
- net at J1.3 (Pin_3), O1.3 (D+): now also JP1.2 (C); no longer R2.2
- new net: JP1.1 (A), R3.2
- new net: JP1.3 (B), R2.2
Other:
- moved on the sheet: J1, O1, R2
